File: idkpad/idkpad.kicad_sch (KiCad schematic)
At the start: 0 parts

Commit message: footprints
Parts:
- added C1, C2: 12p, CC0603JRNPO9BN220:CAPC1608X90, symbol Device:C_Small
- added D1, D10, D11, D12, D13, D14, D15, D16, D17, D18, D2, D3, D4, D5, D6, D7, D8, D9: D, ul_1n4148:SOD123_DIO, symbol Device:D
- added Display1: nice!view, niceview:nice_view, symbol nice:nice!view
- added J1: Conn_01x02_Pin, Connector_JST:JST_PH_S2B-PH-K_1x02_P2.00mm_Horizontal, symbol Connector:Conn_01x02_Pin
- added J2: USB_C_Receptacle_USB2.0_16P, Connector_USB:USB_C_Receptacle_HRO_TYPE-C-31-M-12, symbol Connector:USB_C_Receptacle_USB2.0_16P
- added R1, R2: 22, Resistor_SMD:R_1206_3216Metric_Pad1.30x1.75mm_HandSolder, symbol Device:R
- added R3: R, Resistor_SMD:R_1206_3216Metric_Pad1.30x1.75mm_HandSolder, symbol Device:R
- added R4, R5: 5k1, Resistor_SMD:R_1206_3216Metric_Pad1.30x1.75mm_HandSolder, symbol Device:R_Small
- added SW1, SW10, SW11, SW12, SW13, SW14, SW15, SW16, SW18, SW2, SW3, SW4, SW5, SW6, SW7, SW8, SW9: SW_DIP_x01, kailh:Kailh_socket_MX, symbol Switch:SW_DIP_x01
- added SW17, SW19: RotaryEncoder_Switch, Rotary_Encoder:RotaryEncoder_Alps_EC12E-Switch_Vertical_H20mm, symbol Device:RotaryEncoder_Switch
- added U1: ESP32-C3, esp32-c3:QFN50P500X500X90-33N, symbol esp32:ESP32-C3
- added U2: AMS1117-3.3, Package_TO_SOT_SMD:SOT-223-3_TabPin2, symbol Regulator_Linear:AMS1117-3.3
- added U3: USB6B1, Package_SO:SOIC-8_3.9x4.9mm_P1.27mm, symbol Power_Protection:USB6B1
- added Y1: Crystal_GND24_Small, NX3225GA:OSCCC320X250X90N, symbol Device:Crystal_GND24_Small
Connections:
- new net: D8.2 (A), SW8.1
- new net: C1.1, C2.1
- new net: C1.2, U1.29 (XTAL_N), Y1.3
- new net: D14.2 (A), SW14.1
- new net: R2.1, U1.26 (GPIO19/USB_D+)
- new net: D2.2 (A), SW2.1
- new net: U3.1 (VBUS), U3.8 (VBUS)
- new net: J2.A7 (D-), J2.B7 (D-), U3.2 (I/O1)
- new net: J2.A6 (D+), J2.B6 (D+), U3.3 (I/O2)
- new net: U3.4 (GND), U3.5 (GND)
- new net: D1.2 (A), SW1.1
- new net: D12.2 (A), SW12.1
- new net: D5.2 (A), SW5.1
- new net: D15.2 (A), SW15.1
- new net: U1.11 (VDD3P3_RTC), U1.17 (VDD3P3_CPU), U1.18 (VDD_SPI), U1.2 (VDD3P3), U1.3 (VDD3P3), U1.31 (VDDA), U1.32 (VDDA), U2.2 (VO)
- new net: J1.1 (Pin_1), U2.3 (VI)
- new net: R3.2, SW18.2, U1.7 (CHIP_EN)
- new net: D13.2 (A), SW13.1
- new net: D18.2 (A), SW19.S2
- new net: D3.2 (A), SW3.1
- new net: C2.2, U1.30 (XTAL_P), Y1.1
- new net: D9.2 (A), SW9.1
- new net: D4.2 (A), SW4.1
- new net: D17.2 (A), SW17.S2
- new net: R1.1, U1.25 (GPIO18/USB_D-)
- new net: D16.2 (A), SW16.1
- new net: D11.2 (A), SW11.1
- new net: D7.2 (A), SW7.1
- new net: D6.2 (A), SW6.1
- new net: J2.A5 (CC1), R4.1
- new net: J2.B5 (CC2), R5.1
- new net: D10.2 (A), SW10.1
- new net C1: SW1.2, SW13.2, SW5.2, SW9.2, U1.9 (GPIO4/MTMS)
- new net C2: SW10.2, SW14.2, SW2.2, SW6.2, U1.10 (GPIO5/MTDI)
- new net C3: SW11.2, SW15.2, SW3.2, SW7.2, U1.12 (GPIO6/MTCK)
- new net C4: D1.1 (K), D10.1 (K), D11.1 (K), D12.1 (K), D13.1 (K), D14.1 (K), D15.1 (K), D16.1 (K), D17.1 (K), D18.1 (K), D2.1 (K), D3.1 (K), D4.1 (K), D5.1 (K), D6.1 (K), D7.1 (K), D8.1 (K), D9.1 (K), SW12.2, SW16.2, SW4.2, SW8.2, U1.13 (GPIO7/MTDO), U1.4 (GPIO0/XTAL_32K_P), U1.5 (GPIO1/XTAL_32K_N), U1.6 (GPIO2), U1.8 (GPIO3)
- new net C5: SW17.S1, U1.14 (GPIO8)
- new net C6: SW19.S1, U1.15 (GPIO9)
- new net CS: Display1.5 (CS), U1.16 (GPIO10)
- new net D+: R2.2, U3.6 (I/O2)
- new net D-: R1.2, U3.7 (I/O1)
- new net GND: Display1.4 (GND), J1.2 (Pin_2), J2.A1 (GND), J2.A12 (GND), J2.B1 (GND), J2.B12 (GND), R4.2, R5.2, SW17.C, SW18.1, SW19.C, U1.33 (GND), U2.1 (GND), Y1.4
- new net MOSI: Display1.1 (MOSI), U1.21 (GPIO14/SPICS0)
- new net RE_A1: SW17.A, U1.22 (GPIO15/SPICLK)
- new net RE_A2: SW19.A, U1.24 (GPIO17/SPIQ)
- new net RE_B1: SW17.B, U1.23 (GPIO16/SPID)
- new net RE_B2: SW19.B, U1.27 (GPIO20/U0RXD)
- new net SCK: Display1.2 (SCK), U1.20 (GPIO13/SPIWP)
- new net VBUS: J2.A4 (VBUS), J2.A9 (VBUS), J2.B4 (VBUS), J2.B9 (VBUS), R3.1
- new net VCC: Display1.3 (VCC), U1.19 (GPIO12/SPIHD)
- no-connect marks 0 -> 3

Commit message: prewiring
Parts:
- removed D12, D16, D3, D4, D8: D, ul_1n4148:SOD123_DIO, symbol Device:D
- removed SW12, SW16, SW3, SW4, SW8: SW_DIP_x01, kailh:Kailh_socket_MX, symbol Switch:SW_DIP_x01
- renumbered SW18 to SW3
Connections:
- net C3: now also D1.1 (K), D10.1 (K), D11.1 (K), D13.1 (K), D14.1 (K), D15.1 (K), D17.1 (K), D18.1 (K), D2.1 (K), D5.1 (K), D6.1 (K), D7.1 (K), D9.1 (K), U1.4 (GPIO0/XTAL_32K_P), U1.5 (GPIO1/XTAL_32K_N), U1.6 (GPIO2), U1.8 (GPIO3)
- net C4: now also SW17.S1; no longer D1.1 (K), D10.1 (K), D11.1 (K), D13.1 (K), D14.1 (K), D15.1 (K), D17.1 (K), D18.1 (K), D2.1 (K), D5.1 (K), D6.1 (K), D7.1 (K), D9.1 (K), U1.4 (GPIO0/XTAL_32K_P), U1.5 (GPIO1/XTAL_32K_N), U1.6 (GPIO2), U1.8 (GPIO3)
- net C5: now also SW19.S1; no longer SW17.S1
- net C6: no longer names the net of U1.15 (GPIO9)
- net C6: no longer SW19.S1

Commit message: i forgot to save
Connections:
- net GND: now also U3.4 (GND), U3.5 (GND)
- net VBUS: now also U3.1 (VBUS), U3.8 (VBUS)
Changed lines of the file:
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@@
+	)
+	(symbol
+		(lib_id "power:VBUS")
+		(at 63.5 49.53 0)
+		(unit 1)
+		(exclude_from_sim no)
+		(in_bom yes)
+		(on_board yes)
+		(dnp no)
+		(fields_autoplaced yes)
+		(property "Reference" "#PWR014"
+			(at 63.5 53.34 0)
+			(effects
+				(font
+					(size 1.27 1.27)
+				)
+				(hide yes)
+			)
+		)
+		(property "Value" "VBUS"
+			(at 63.5 44.45 0)
+			(effects
+				(font
+					(size 1.27 1.27)
+				)
+			)
+		)
+		(property "Footprint" ""
+			(at 63.5 49.53 0)
+			(effects
+				(font
+					(size 1.27 1.27)
+				)
+				(hide yes)
+			)
+		)
+		(property "Datasheet" ""
+			(at 63.5 49.53 0)
+			(effects
+				(font
+					(size 1.27 1.27)
+				)
+				(hide yes)
+			)
+		)
+		(property "Description" "Power symbol creates a global label with name \"VBUS\""
+			(at 63.5 49.53 0)
+			(effects
+				(font
+					(size 1.27 1.27)
+				)
+				(hide yes)
+			)
+		)
+		(pin "1"
+		)
+		(instances
+			(project ""
+				(path "/2745bbf1-7cb1-4bf2-b802-d8e257ca52fa"
+					(reference "#PWR014")
+					(unit 1)
+				)
+			)
+		)
 	)
 	(symbol
@@
 					(unit 1)
 				)
+			)
+		)
+	)
+	(symbol
+		(lib_id "power:GND")
+		(at 63.5 64.77 0)
+		(unit 1)
+		(exclude_from_sim no)
+		(in_bom yes)
+		(on_board yes)
+		(dnp no)
+		(fields_autoplaced yes)
+		(property "Reference" "#PWR013"
+			(at 63.5 71.12 0)
+			(effects
+				(font
+					(size 1.27 1.27)
+				)
+				(hide yes)
+			)
+		)
+		(property "Value" "GND"
+			(at 63.5 69.85 0)
+			(effects
+				(font
+					(size 1.27 1.27)
+				)
+			)
+		)
+		(property "Footprint" ""
+			(at 63.5 64.77 0)
+			(effects
+				(font
+					(size 1.27 1.27)
+				)
+				(hide yes)
+			)
+		)
+		(property "Datasheet" ""
+			(at 63.5 64.77 0)
+			(effects
+				(font
+					(size 1.27 1.27)
+				)
+				(hide yes)
+			)
+		)
+		(property "Description" "Power symbol creates a global label with name \"GND\" , ground"
+			(at 63.5 64.77 0)
+			(effects
+				(font
+					(size 1.27 1.27)
+				)
+				(hide yes)
+			)
+		)
+		(pin "1"
+		)
+		(instances
+			(project ""
+				(path "/2745bbf1-7cb1-4bf2-b802-d8e257ca52fa"
+					(reference "#PWR013")
+					(unit 1)
+				)
